File: pcbs/sandwichCircuit/sandwichCircuit.kicad_pcb (KiCad board)
At the start: 2 copper layers, 0 parts

Commit message: Progress sandwhich board
Parts:
- added J1: Conn_01x19_Pin, Connector_PinHeader_2.54mm:PinHeader_1x19_P2.54mm_Vertical, F.Cu at (136.7, 59.9)
- added U1: ESP32-DevKitC, Espressif:ESP32-DevKitC, F.Cu at (87.4, 59.9)
Other:
- net class Default removed
