File: pcbs/hautDeForme/hautDeForme.kicad_pcb (KiCad board)
At the start: 2 copper layers, 29.8 x 68.3 mm, 40 parts, among them J1 Conn_02x07_Counter_Clockwise, J6 USB4105-GF-A, U2 AZ1117CH-3.3TRG1, U4 CP2102N

Commit message: Haut de forme v0.1
Parts:
- 3V1, 5V1, TP1, TP2, TP3, TP4, TP5: moved to F.Cu
- moved TP5 30.9 mm to (122.7, 104.2), turned to 0 degrees
- moved TP1 25.2 mm to (122.7, 107.7), turned to 0 degrees
- moved TP2 25.2 mm to (122.7, 111.3), turned to 0 degrees
- moved TP4 23.7 mm to (125.5, 111.3), turned to 0 degrees
- moved D6 17.9 mm to (138.8, 111.4)
- moved R6 17.9 mm to (140.7, 111.4)
- moved JP2 17.6 mm to (133.8, 105.1), turned to 90 degrees
- moved JP3 15.6 mm to (128.8, 105.1), turned to 90 degrees
- moved C16 14.1 mm to (139.9, 141.4)
- moved TP3 11.7 mm to (139.7, 107.7), turned to 0 degrees
- moved C15 10.5 mm to (136.2, 143.1)
- moved D14 8.64 mm to (139.7, 143.8)
- moved 5V1 6.00 mm to (124.1, 128.7), turned to 0 degrees
- moved JP1 5.04 mm to (131.8, 139.8), turned to 180 degrees
- moved C6 3.74 mm to (125.5, 125.8)
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Routing:
- net +3.3V: track 7.55 -> 95.1 mm, vias 0 -> 7
- net TX: track 0.00 -> 46.9 mm
- net IO5: track 0.00 -> 46.9 mm, vias 0 -> 2
- net RX: track 0.00 -> 40.1 mm
- net +5V: track 7.50 -> 33.2 mm, vias 0 -> 2
- net RST: track 0.00 -> 17.5 mm
- net IO23: track 0.00 -> 16.1 mm
- net IO18: track 0.00 -> 14.5 mm, vias 0 -> 1
- net IO0: track 0.00 -> 12.9 mm
- net RX0: track 0.00 -> 10.9 mm, vias 0 -> 1
- net TX0: track 0.00 -> 10.9 mm, vias 0 -> 1
- net /CP2102_1/DCD: track 1.68 -> 9.70 mm
- net IO19: track 0.00 -> 7.15 mm
- net IO21: track 0.00 -> 6.52 mm
- net IO22: track 0.00 -> 4.97 mm
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- added copper zone on B.Cu, net +5V
- added copper zone on B.Cu, net GND
- added copper zone on F.Cu, net GND
Other:
- outline, holes or cut-outs redrawn
- board text added: "(c) ${COMPANY} - ${ISSUE_DATE} ${TITLE} - rev ${REVISION}"
- board text added: "3V3"
- board text added: "5V"
- board text added: "CONN OK"
- board text added: "DCD"
- board text added: "IO0"
- board text added: "IO18"
- board text added: "IO19"
- board text added: "IO21"
- board text added: "IO22"
- board text added: "IO5"
- board text added: "POWER OK"
- board text added: "RST"
- board text added: "RX"
- board text added: "RX0"
- board text added: "TX"
- board text added: "TX0"
