File: pcbs/hautDeForme/CP2102.kicad_sch (KiCad schematic)
At the start: 12 parts, among them U3 CP2102N

Commit message: Haut de forme v0.1
Parts:
- renumbered R15 to R23, R16 to R24, U3 to U4
Other:
- title: CP2102 28Pin Auxiliary circuit -> Haut de Forme
Changed lines of the file:
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@@
   (paper "A4")
   (title_block
-    (title "CP2102 28Pin Auxiliary circuit")
-    (date "2025-03-01")
-    (rev "0.2.0")
+    (title "Haut de Forme")
+    (date "2025-03-03")
+    (rev "0.1.0")
     (company "Martin Roger")
   )
@@
   (symbol (lib_id "Device:R_Small") (at 107.95 86.36 90) (unit 1)
     (in_bom yes) (on_board yes) (dnp no) (fields_autoplaced)
-    (property "Reference" "R15" (at 107.95 81.28 90)
+    (property "Reference" "R23" (at 107.95 81.28 90)
       (effects (font (size 1.27 1.27)))
     )
@@
   (symbol (lib_id "Device:R_Small") (at 113.03 95.25 0) (unit 1)
     (in_bom yes) (on_board yes) (dnp no) (fields_autoplaced)
-    (property "Reference" "R16" (at 115.57 94.615 0)
+    (property "Reference" "R24" (at 115.57 94.615 0)
       (effects (font (size 1.27 1.27)) (justify left))
     )
@@
   (symbol (lib_id "Interface_USB:CP2102N-Axx-xQFN28") (at 153.67 101.6 0) (unit 1)
     (in_bom yes) (on_board yes) (dnp no) (fields_autoplaced)
-    (property "Reference" "U3" (at 155.6259 134.62 0)
+    (property "Reference" "U4" (at 155.6259 134.62 0)
       (effects (font (size 1.27 1.27)) (justify left))
     )

Commit message: Projects consistency update
Parts:
- renumbered C8 to C13, C8 to C14, D2 to D11, D1 to D9, R4 to R25, R4 to R26, R4 to R27, R1 to R34, R2 to R35
