File: pcbs/hautDeForme/USBC.kicad_sch (KiCad schematic)
At the start: 7 parts, among them J5 USB4105-GF-A

Commit message: Haut de forme v0.1
Parts:
- renumbered D10 to D14, J5 to J6, R20 to R28, R22 to R30
Other:
- title: (none) -> Haut de Forme
Changed lines of the file:
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@@
   (paper "A4")
   (title_block
-    (date "2025-03-01")
-    (rev "0.2.0")
+    (title "Haut de Forme")
+    (date "2025-03-03")
+    (rev "0.1.0")
     (company "Martin Roger")
   )
@@
   (symbol (lib_id "USB4105-GF-A:USB4105-GF-A") (at 85.09 58.42 0) (unit 1)
     (in_bom yes) (on_board yes) (dnp no) (fields_autoplaced)
-    (property "Reference" "J5" (at 85.09 41.91 0)
+    (property "Reference" "J6" (at 85.09 41.91 0)
       (effects (font (size 1.27 1.27)))
     )
@@
   (symbol (lib_id "Device:R_Small") (at 123.19 55.88 90) (unit 1)
     (in_bom yes) (on_board yes) (dnp no) (fields_autoplaced)
-    (property "Reference" "R22" (at 123.19 50.8 90)
+    (property "Reference" "R30" (at 123.19 50.8 90)
       (effects (font (size 1.27 1.27)))
     )
@@
   (symbol (lib_id "SamacSys_Parts:1N5819HW-7-F") (at 176.53 33.02 180) (unit 1)
     (in_bom yes) (on_board yes) (dnp no) (fields_autoplaced)
-    (property "Reference" "D10" (at 168.91 26.67 0)
+    (property "Reference" "D14" (at 168.91 26.67 0)
       (effects (font (size 1.27 1.27)))
     )
@@
   (symbol (lib_id "Device:R_Small") (at 59.69 53.34 90) (unit 1)
     (in_bom yes) (on_board yes) (dnp no) (fields_autoplaced)
-    (property "Reference" "R20" (at 59.69 48.26 90)
-      (effects (font (size 1.27 1.27)))
-    )
+    (property "Reference" "R28" (at 59.69 48.26 90)
+      (effects (font (size 1.27 1.27)))
+    )

Commit message: Projects consistency update
Parts:
- D14: footprint Diode_SMD:D_SOD-123 -> DIY:SOD3716X145N; symbol SamacSys_Parts:1N5819HW-7-F -> DIY:1N5819HW-7-F
- J6: symbol USB4105-GF-A:USB4105-GF-A -> DIY:USB4105-GF-A
- renumbered C8 to C15, D15 to D8, R4 to R29
