File: pcbs/hautDeForme/hautDeForme.kicad_sch (KiCad schematic)
At the start: 21 parts, among them J1 Conn_02x07_Counter_Clockwise, U2 AZ1117CH-3.3TRG1

Commit message: Haut de forme v0.1
Parts:
- J1: now not fitted; now left out of the parts list
Other:
- title: A1S Mini Board -> Haut de Forme
Changed lines of the file:
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@@
   (paper "A4")
   (title_block
-    (title "A1S Mini Board")
-    (date "2025-03-01")
-    (rev "0.2.0")
+    (title "Haut de Forme")
+    (date "2025-03-03")
+    (rev "0.1.0")
     (company "Martin Roger")
   )
@@
   )
   (symbol (lib_id "Connector_Generic:Conn_02x07_Odd_Even") (at 124.46 104.14 0) (unit 1)
-    (in_bom yes) (on_board yes) (dnp no)
+    (in_bom no) (on_board yes) (dnp yes)
     (property "Reference" "J1" (at 125.73 91.44 0)
       (effects (font (size 1.27 1.27)))

Commit message: Move to CP2102 non N
Other:
- sheet CP2102_1: file CP2102.kicad_sch -> CP2102-GM.kicad_sch
Changed lines of the file:
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@@
 	(title_block
 		(title "Haut de Forme")
-		(date "2025-03-11")
-		(rev "0.1.1")
+		(date "2025-05-26")
+		(rev "0.2.0")
 		(company "Martin Roger")
 	)
@@
 			)
 		)
-		(property "Sheetfile" "CP2102.kicad_sch"
+		(property "Sheetfile" "CP2102-GM.kicad_sch"
 			(at 265.43 114.3 90)
 			(effects
