File: pcbs/AiO-i2s-DAC/CP2102.kicad_sch (KiCad schematic)
At the start: 12 parts, among them U3 CP2102N

Commit message: Exposing DCD, 3V3 and 5V in schematic
Other:
- title: A1S Mini Board -> AiO-i2s-DAC
Changed lines of the file:
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@@
 	(paper "A4")
 	(title_block
-		(title "A1S Mini Board")
-		(date "2025-03-30")
-		(rev "0.3.0")
+		(title "AiO-i2s-DAC")
+		(date "2025-05-18")
+		(rev "0.1.2")
 		(company "Martin Roger")
 	)
