File: pcbs/AiO-i2s-DAC/AiO-i2s-DAC.kicad_pcb (KiCad board)
At the start: 2 copper layers, 58.8 x 55.7 mm, 85 parts, among them J1 UART1, J2 SJ-3524-SMT-TR-PI, J3 Audio Out, J4 UART0, J5 USB4105-GF-A, J6 USB4105-GF-A, Q3 BC818, Q4 MBT3904DW1, Q6 MBT3904DW1, U1 ESP32 A1S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

Commit message: Footprints update
Parts:
- removed C4, C5: 0.1uF 50V, Capacitor_SMD:C_0603_1608Metric
- removed R10, R11, R31: 0R, Resistor_SMD:R_0603_1608Metric
- removed R8, R9: 22R 1%, Resistor_SMD:R_0603_1608Metric
- added C17: 2.2uF 16V, Capacitor_SMD:C_0603_1608Metric, F.Cu at (98.0, 73.1)
- added C18: 0.1uF 50V, Capacitor_SMD:C_0603_1608Metric, F.Cu at (98.0, 75.6)
- added C20: 2.2uF 16V, Capacitor_SMD:C_0603_1608Metric, F.Cu at (98.0, 78.2)
- added C21: 10uF 16V, Capacitor_SMD:C_0805_2012Metric, F.Cu at (98.2, 88.4)
- added C22: 0.1uF 50V, Capacitor_SMD:C_0603_1608Metric, F.Cu at (98.0, 80.7)
- added C23: 0.1uF 50V, Capacitor_SMD:C_0603_1608Metric, F.Cu at (98.0, 83.2)
- added C24: 10uF 16V, Capacitor_SMD:C_0805_2012Metric, F.Cu at (98.2, 91.5)
- added C25: 0.1uF 50V, Capacitor_SMD:C_0603_1608Metric, F.Cu at (98.0, 85.7)
- added C26: 10uF 16V, Capacitor_SMD:C_0805_2012Metric, F.Cu at (98.2, 94.5)
- added C27: 2.2nF, Capacitor_SMD:C_0603_1608Metric, F.Cu at (102.0, 73.1)
- added C28: 2.2nF, Capacitor_SMD:C_0603_1608Metric, F.Cu at (102.0, 75.6)
- added C29: 10uF 16V, Capacitor_SMD:C_0805_2012Metric, F.Cu at (98.2, 97.5)
- added J7: Conn_01x02, Connector_PinHeader_2.54mm:PinHeader_1x02_P2.54mm_Vertical, F.Cu at (102.8, 89.3)
- added J8: Conn_01x02, Connector_PinHeader_2.54mm:PinHeader_1x02_P2.54mm_Vertical, F.Cu at (107.4, 89.3)
- added JP3: SolderJumper_2_Bridged, Jumper:SolderJumper-2_P1.3mm_Bridged_RoundedPad1.0x1.5mm, F.Cu at (98.2, 100.8)
- added R3: 470R 1%, Resistor_SMD:R_0603_1608Metric, F.Cu at (102.0, 78.2)
- added R36: 10K 1%, Resistor_SMD:R_0603_1608Metric, F.Cu at (102.0, 83.2)
- added R37: 10K 1%, Resistor_SMD:R_0603_1608Metric, F.Cu at (102.0, 85.7)
- added R38: 10K 1%, Resistor_SMD:R_0603_1608Metric, F.Cu at (106.0, 73.1)
- added R39: 10K 1%, Resistor_SMD:R_0603_1608Metric, F.Cu at (106.0, 75.6)
- added R4: 470R 1%, Resistor_SMD:R_0603_1608Metric, F.Cu at (102.0, 80.7)
- added R40: 10K 1%, Resistor_SMD:R_0603_1608Metric, F.Cu at (106.0, 78.2)
- added R41: 0R, Resistor_SMD:R_0603_1608Metric, F.Cu at (106.0, 80.7)
- added U5: PCM5102A, Package_SO:TSSOP-20_4.4x6.5mm_P0.65mm, F.Cu at (105.2, 98.2)
- J1: footprint Connector_PinHeader_2.54mm:PinHeader_1x04_P2.54mm_Vertical -> Connector_PinHeader_2.54mm:PinHeader_1x05_P2.54mm_Vertical
- J2: value SJ-3524-SMT-TR-PI -> SJ-3524-SMT-TR
- JP1: value SolderJumper_3_Bridged12 -> ActDCD
- JP2: value SolderJumper_2_Bridged -> SIL_BOOT
- U1: value ESP32 A1S -> ESP32-WROVER-E; footprint DIY:ESP32-A1S -> PCM_Espressif:ESP32-WROVER-E_ThermalVias
- moved U1 18.4 mm to (146.8, 96.8)
- moved GND1 3.20 mm to (150.7, 131.1)
- moved J1 2.55 mm to (146.8, 131.7)
Connections:
- C1 pad 1: GND -> AGND
- C10 pad 1: GND -> AGND
- C11 pad 1: GND -> AGND
- C12 pad 1: GND -> AGND
- C13 pad 1: GND -> AGND
- C14 pad 1: GND -> AGND
- C15 pad 1: GND -> AGND
- C16 pad 1: GND -> AGND
- C2 pad 1: GND -> AGND
- C3 pad 1: GND -> AGND
- C6 pad 1: GND -> AGND
- C7 pad 1: GND -> AGND
- C8 pad 1: GND -> AGND
- C9 pad 1: GND -> AGND
- D5 pad 1: GND -> AGND
- D7 pad 1: GND -> AGND
- D8 pad 1: GND -> AGND
- GND1 pad 1: GND -> AGND
- H1 pad 1: GND -> AGND
- H2 pad 1: GND -> AGND
- H3 pad 1: GND -> AGND
- H4 pad 1: GND -> AGND
- J1 pad 1: GND -> AGND
- J1 pad 2: TXD1 -> DCD
- J1 pad 3: RXD1 -> TXD1
- J1 pad 4: +3.3V -> RXD1
- J4 pad 1: GND -> AGND
- J5 pad A1_B12: GND -> AGND
- J5 pad B1_A12: GND -> AGND
- J6 pad A1_B12: GND -> AGND
- J6 pad B1_A12: GND -> AGND
- JP1 pad 1: GND -> AGND
- JP1 pad 2: /CP2102_1/DCD -> DCD
- JP2 pad 2: GND -> AGND
- Q4 pad 1: GND -> AGND
- Q4 pad 4: GND -> AGND
- R16 pad 2: GND -> AGND
- R20 pad 1: GND -> AGND
- R21 pad 2: GND -> AGND
- R22 pad 2: GND -> AGND
- R24 pad 2: GND -> AGND
- R28 pad 1: GND -> AGND
- R29 pad 2: GND -> AGND
- R30 pad 2: GND -> AGND
- S2 pad 1: GND -> AGND
- S2 pad 2: GND -> AGND
- U1 pad 1: GND -> AGND
- U1 pad 10: Net-(JP2-A) -> WSEL
- U1 pad 11: IO2 -> DIN
- U1 pad 12: unconnected-(U1-IO4-Pad12) -> BCLK
- U1 pad 15: unconnected-(U1-MIC2P-Pad15) -> AGND
- U1 pad 17: unconnected-(U1-MIC1P-Pad17) -> (no net)
- U1 pad 18: unconnected-(U1-MIC2N-Pad18) -> (no net)
- U1 pad 19: GND -> (no net)
- U1 pad 20: GND -> (no net)
- U1 pad 21: unconnected-(U1-LINEINR-Pad21) -> (no net)
- U1 pad 22: unconnected-(U1-LINEINL-Pad22) -> (no net)
- U1 pad 23: unconnected-(U1-SPORP-Pad23) -> Net-(JP2-A)
- U1 pad 24: unconnected-(U1-SPORN-Pad24) -> IO2
- U1 pad 25: unconnected-(U1-SPOLP-Pad25) -> IO0
- U1 pad 27: HPOUTL -> (no net)
- U1 pad 28: HPOUTR -> (no net)
- U1 pad 3: unconnected-(U1-SENSOR_VN-Pad3) -> EN
- U1 pad 31: unconnected-(U1-IO23-Pad31) -> RXD1
- U1 pad 32: RXD1 -> (no net)
- U1 pad 34: unconnected-(U1-IO21-Pad34) -> RXD0
- U1 pad 35: EN -> TXD0
- U1 pad 36: TXD0 -> unconnected-(U1-GPIO22-Pad36)
- U1 pad 37: RXD0 -> unconnected-(U1-GPIO23-Pad37)
- U1 pad 38: GND -> AGND
- U1 pad 39: GND -> AGND
- U1 pad 6: IO0 -> unconnected-(U1-GPIO34/ADC1_CH6-Pad6)
- U2 pad 1: GND -> AGND
- U3 pad 29: GND -> AGND
- U3 pad 3: GND -> AGND
- U4 pad 1: /CP2102_1/DCD -> DCD
- U4 pad 29: GND -> AGND
- U4 pad 3: GND -> AGND
Routing:
- net HPOUTR: track 35.1 -> 0.00 mm
- net HPOUTL: track 25.5 -> 0.00 mm
- net DCD: track 0.00 -> 16.6 mm, vias 0 -> 1
- net /CP2102_1/DCD: track 16.6 -> 0.00 mm, vias 1 -> 0
- net Net-(C5-Pad1): track 1.80 -> 0.00 mm
- net Net-(C4-Pad1): track 1.80 -> 0.00 mm
- net TXD1: track 58.2 -> 59.4 mm
- net IO18: track 25.1 -> 24.2 mm
- net RXD1: track 68.4 -> 67.5 mm
- net GND: vias 304 -> 0
- net AGND: vias 1 -> 303
- added copper zone on B.Cu, net AGND
- added copper zone on F.Cu, net AGND
- removed copper zone on B.Cu, net GND
- removed copper zone on F.Cu, net GND

Commit message: Pre-layout
Parts:
- moved C28 93.1 mm to (177.2, 130.7), turned to -90 degrees
- moved C27 89.8 mm to (170.9, 130.7), turned to -90 degrees
- moved R4 88.8 mm to (175.4, 130.7), turned to -90 degrees
- moved R3 85.2 mm to (169.2, 130.7), turned to 90 degrees
- moved C17 83.1 mm to (157.6, 131.1), turned to 90 degrees
- moved R38 80.2 mm to (163.1, 129.5), turned to -90 degrees
- moved C22 79.9 mm to (160.5, 130.4), turned to 180 degrees
- moved C21 76.4 mm to (160.8, 132.4)
- moved C18 73.4 mm to (156.2, 120.5)
- moved C20 73.3 mm to (153.3, 126.3), turned to 90 degrees
- moved R40 73.2 mm to (163.2, 123.8)
- moved R36 72.0 mm to (163.3, 121.0)
- moved C25 72.0 mm to (154.6, 130.3)
- moved R37 69.9 mm to (163.3, 119.3)
- moved C26 67.7 mm to (154.3, 132.4), turned to 180 degrees
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Routing:
- net AGND: track 30.3 -> 0.00 mm, vias 303 -> 230
- net EN: track 51.2 -> 22.7 mm, vias 4 -> 0
- net DCD: track 16.6 -> 42.7 mm, vias 1 -> 2
- net LOUT: track 20.8 -> 0.00 mm, vias 1 -> 0
- net ROUT: track 19.2 -> 0.00 mm, vias 1 -> 0
- net IO2: track 21.3 -> 32.8 mm, vias 2 -> 4
- net IO0: track 28.9 -> 34.1 mm, vias 2 -> 4
- net +3.3V: track 151.9 -> 155.5 mm
- net IO5: track 22.7 -> 19.7 mm
- net RXD0: track 38.9 -> 40.9 mm
- net RXD1: track 67.5 -> 66.2 mm
- net IO18: track 24.2 -> 25.3 mm, vias 0 -> 2
- net TXD0: track 37.5 -> 38.2 mm

Commit message: CP2102 instead of CP2102N
Moving some components to CP2102 non N
Parts:
- removed J8: Conn_01x02, Connector_PinHeader_2.54mm:PinHeader_1x02_P2.54mm_Vertical
- added FB1: 120R@100MHz, Inductor_SMD:L_0603_1608Metric, F.Cu at (151.7, 131.6)
- JP3: value SolderJumper_2_Bridged -> Ferrite bypass; footprint Jumper:SolderJumper-2_P1.3mm_Bridged_RoundedPad1.0x1.5mm -> Jumper:SolderJumper-2_P1.3mm_Open_RoundedPad1.0x1.5mm
- U4: value CP2102N -> CP2102-GM
- moved J7 73.1 mm to (171.2, 115.1), turned to 90 degrees
- moved J3 5.46 mm to (182.7, 115.1)
- moved D11 3.30 mm to (160.9, 110.2)
- moved D9 3.30 mm to (160.9, 106.9)
- moved R34 3.30 mm to (159.1, 106.9), turned to 90 degrees
- moved R35 3.30 mm to (159.1, 110.2), turned to -90 degrees
- moved J2 2.75 mm to (179.5, 122.7)
- moved R36 2.05 mm to (164.3, 119.3)
- moved R37 1.94 mm to (164.3, 120.9)
- moved C21 1.14 mm to (161.9, 132.5)
- moved C25 1.14 mm to (155.7, 130.4)
- moved C26 1.14 mm to (155.4, 132.5)
- moved R38 1.14 mm to (164.2, 129.6)
- moved C24 1.14 mm to (152.4, 121.2)
- moved C29 1.14 mm to (157.2, 118.6)
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Connections:
- net /CP2102_1/CTS renamed /CP2102-GM/CTS
- net /CP2102_1/D+ renamed /CP2102-GM/D+
- net /CP2102_1/D- renamed /CP2102-GM/D-
- net /CP2102_1/DSR renamed /CP2102-GM/DSR
- net /CP2102_1/DTR renamed /CP2102-GM/DTR
- net /CP2102_1/RI renamed /CP2102-GM/RI
- net /CP2102_1/RTS renamed /CP2102-GM/RTS
- D11 pad 1: Net-(D11-K) -> TXD1
- D9 pad 1: Net-(D9-K) -> RXD1
- U4 pad 18: Net-(D11-K) -> unconnected-(U4-~{RXT}/GPIO.1-Pad18)
- U4 pad 19: Net-(D9-K) -> unconnected-(U4-~{TXT}/GPIO.0-Pad19)
Routing:
- net BCLK: track 0.00 -> 44.8 mm, vias 0 -> 2
- net WSEL: track 0.00 -> 44.7 mm, vias 0 -> 2
- net DIN: track 0.00 -> 44.4 mm, vias 0 -> 2
- net +3.3V: track 155.5 -> 183.6 mm
- net AVDD: track 0.00 -> 23.1 mm
- net LOUT: track 0.00 -> 19.5 mm
- net ROUT: track 0.00 -> 18.9 mm
- net Net-(U5-OUTR): track 0.00 -> 18.1 mm, vias 0 -> 2
- net Net-(U5-OUTL): track 0.00 -> 14.5 mm, vias 0 -> 2
- net DVDD: track 0.00 -> 6.82 mm
- net MUTE: track 0.00 -> 6.73 mm
- net FORMAT: track 0.00 -> 6.33 mm
- net Net-(U5-CAPM): track 0.00 -> 5.20 mm
- net SCK_IN: track 0.00 -> 5.07 mm
- net Net-(U5-LDOO): track 0.00 -> 4.39 mm
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Other:
- board text added: "UART0 ↑↑"
- board text added: "UART1 to car"
- board text removed: "UART0"
- board text removed: "UART1 To car"
