File: pcbs/AiO-i2s-DAC/AiO-i2s-DAC.kicad_pcb (KiCad board)
At the start: 2 copper layers, 58.8 x 55.7 mm, 102 parts, among them J1 UART1, J2 SJ-3524-SMT-TR, J3 Audio Out, J4 UART0, J5 USB4105-GF-A, J6 USB4105-GF-A, J7 Conn_01x02, Q3 BC818, Q4 MBT3904DW1, Q6 MBT3904DW1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

Commit message: LCSC BOM Preparation
Parts:
- U3: value CP2102N -> CP2102-GM

Commit message: Added board properties
Other:
- board text added: "0.1524 mm / 0.1524 mm"
- board text added: "0.3000 mm"
- board text added: "1.6000 mm"
- board text added: "2"
- board text added: "58.7500 mm x 55.7500 mm"
- board text added: "BOARD CHARACTERISTICS"
- board text added: "Board Thickness:"
- board text added: "Board overall dimensions:"
- board text added: "Castellated pads:"
- board text added: "Copper Finish:"
- board text added: "Copper Layer Count:"
- board text added: "Edge card connectors:"
- board text added: "Impedance Control:"
- board text added: "Min hole diameter:"
- board text added: "Min track/spacing:"
- board text added: "No"
- board text added: "None"
- board text added: "Plated Board Edge:"

Commit message: UART0 LEDs correction
Parts:
- moved D1 3.30 mm to (160.9, 93.6)
- moved D2 3.30 mm to (160.9, 96.9)
- moved R1 3.30 mm to (159.1, 93.6), turned to 90 degrees
- moved R2 3.30 mm to (159.1, 96.9), turned to -90 degrees
Connections:
- D1 pad 1: Net-(D1-K) -> RXD0
- D2 pad 1: Net-(D2-K) -> TXD0
- U3 pad 18: Net-(D2-K) -> unconnected-(U3-~{RXT}/GPIO.1-Pad18)
- U3 pad 19: Net-(D1-K) -> unconnected-(U3-~{TXT}/GPIO.0-Pad19)
Routing:
- net Net-(D1-K): track 2.12 -> 0.00 mm
- net Net-(D2-K): track 2.12 -> 0.00 mm
- net RXD0: track 40.9 -> 42.9 mm
- net TXD0: track 38.2 -> 39.7 mm
- net Net-(D2-A): track 1.79 -> 2.45 mm
- net Net-(D1-A): track 1.79 -> 2.45 mm
Changed lines of the file:
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@@
 	(title_block
 		(title "AiO-i2s-DAC")
-		(date "2025-09-02")
-		(rev "0.1.6")
+		(date "2025-10-05")
+		(rev "0.1.7")
 		(company "Martin Roger")
 	)
@@
 	(net 83 "Net-(Q4B-B2)")
 	(net 84 "Net-(Q4A-B1)")
-	(net 85 "Net-(D2-K)")
+	(net 85 "unconnected-(U3-~{RXT}{slash}GPIO.1-Pad18)")
 	(net 86 "/CP2102-GM/CTS")
 	(net 87 "Net-(D11-A)")
-	(net 88 "Net-(D1-K)")
+	(net 88 "unconnected-(U3-~{TXT}{slash}GPIO.0-Pad19)")
 	(net 89 "Net-(C9-Pad2)")
 	(net 90 "Net-(U5-LDOO)")
@@
 	(footprint "Resistor_SMD:R_0603_1608Metric"
 		(layer "F.Cu")
-		(at 159.131 96.901 -90)
+		(at 159.131 93.599 90)
 		(descr "Resistor SMD 0603 (1608 Metric), square (rectangular) end terminal, IPC_7351 nominal, (Body size source: IPC-SM-782 page 72, https://www.pcb-3d.com/wordpress/wp-content/uploads/ipc-sm-782a_amendment_1_and_2.pdf), generated with kicad-footprint-generator")
 		(tags "resistor")
@@
 		)
 		(property "Datasheet" "https://www.yageo.com/upload/media/product/products/datasheet/rchip/PYu-RC_Group_51_RoHS_L_12.pdf"
-			(at 0 0 270)
+			(at 0 0 90)
 			(layer "F.Fab")
 			(hide yes)
@@
 		)
 		(property "LCSC" "C21190"
-			(at 0 0 270)
+			(at 0 0 90)
 			(unlocked yes)
 			(layer "F.Fab")
@@
 		)
 		(property "LCSC alt" "C22548"
-			(at 0 0 270)
+			(at 0 0 90)
 			(unlocked yes)
 			(layer "F.Fab")
@@
 		(attr smd)
 		(fp_line
-			(start -0.237258 0.5225)
-			(end 0.237258 0.5225)
+			(start -0.237258 -0.5225)
+			(end 0.237258 -0.5225)
 			(stroke
 				(width 0.12)
@@
 		)
 		(fp_line
-			(start -0.237258 -0.5225)
-			(end 0.237258 -0.5225)
+			(start -0.237258 0.5225)
+			(end 0.237258 0.5225)
 			(stroke
 				(width 0.12)
@@
 		)
 		(fp_line
-			(start -1.48 0.73)
-			(end -1.48 -0.73)
+			(start 1.48 -0.73)
+			(end 1.48 0.73)
 			(stroke
 				(width 0.05)
@@
 		)
 		(fp_line
-			(start 1.48 0.73)
-			(end -1.48 0.73)
+			(start -1.48 -0.73)
+			(end 1.48 -0.73)
 			(stroke
 				(width 0.05)
@@
 		)
 		(fp_line
-			(start -1.48 -0.73)
-			(end 1.48 -0.73)
+			(start 1.48 0.73)
+			(end -1.48 0.73)
 			(stroke
 				(width 0.05)
@@
 		)
 		(fp_line
-			(start 1.48 -0.73)
-			(end 1.48 0.73)
+			(start -1.48 0.73)
+			(end -1.48 -0.73)
 			(stroke
 				(width 0.05)
@@
 		)
 		(fp_line
-			(start -0.8 0.4125)
-			(end -0.8 -0.4125)
+			(start 0.8 -0.4125)
+			(end 0.8 0.4125)
 			(stroke
 				(width 0.1)
@@
 		)
 		(fp_line
-			(start 0.8 0.4125)
-			(end -0.8 0.4125)
+			(start -0.8 -0.4125)
+			(end 0.8 -0.4125)
 			(stroke
 				(width 0.1)
@@
 		)
 		(fp_line
-			(start -0.8 -0.4125)
-			(end 0.8 -0.4125)
+			(start 0.8 0.4125)
+			(end -0.8 0.4125)
 			(stroke
 				(width 0.1)
@@
 		)
 		(fp_line
-			(start 0.8 -0.4125)
-			(end 0.8 0.4125)
+			(start -0.8 0.4125)
+			(end -0.8 -0.4125)
 			(stroke
 				(width 0.1)
@@
 		)
 		(pad "1" smd roundrect
-			(at -0.825 0 270)
+			(at -0.825 0 90)
 			(size 0.8 0.95)
 			(layers "F.Cu" "F.Mask" "F.Paste")
@@
 		)
 		(pad "2" smd roundrect
-			(at 0.825 0 270)
+			(at 0.825 0 90)
 			(size 0.8 0.95)
 			(layers "F.Cu" "F.Mask" "F.Paste")
@@
 			(layers "F.Cu" "F.Mask" "F.Paste")
 			(roundrect_rratio 0.25)
-			(net 85 "Net-(D2-K)")
+			(net 85 "unconnected-(U3-~{RXT}{slash}GPIO.1-Pad18)")
 			(pinfunction "~{RXT}/GPIO.1")
-			(pintype "bidirectional")
+			(pintype "bidirectional+no_connect")
 		)
 		(pad "19" smd roundrect
@@
 			(layers "F.Cu" "F.Mask" "F.Paste")
 			(roundrect_rratio 0.25)
-			(net 88 "Net-(D1-K)")
+			(net 88 "unconnected-(U3-~{TXT}{slash}GPIO.0-Pad19)")
 			(pinfunction "~{TXT}/GPIO.0")
-			(pintype "bidirectional")
+			(pintype "bidirectional+no_connect")
 		)
 		(pad "20" smd roundrect
@@
 	(footprint "Resistor_SMD:R_0603_1608Metric"
 		(layer "F.Cu")
-		(at 159.131 93.599 90)
+		(at 159.131 96.901 -90)
 		(descr "Resistor SMD 0603 (1608 Metric), square (rectangular) end terminal, IPC_7351 nominal, (Body size source: IPC-SM-782 page 72, https://www.pcb-3d.com/wordpress/wp-content/uploads/ipc-sm-782a_amendment_1_and_2.pdf), generated with kicad-footprint-generator")
 		(tags "resistor")
@@
 		)
 		(property "LCSC" "C21190"
-			(at 0 0 90)
+			(at 0 0 270)
 			(unlocked yes)
 			(layer "F.Fab")
@@
 		)
 		(property "LCSC alt" "C22548"
-			(at 0 0 90)
+			(at 0 0 270)
 			(unlocked yes)
 			(layer "F.Fab")
@@
 		(attr smd)
 		(fp_line
-			(start -0.237258 -0.5225)
-			(end 0.237258 -0.5225)
+			(start -0.237258 0.5225)
+			(end 0.237258 0.5225)
 			(stroke
 				(width 0.12)
@@
 		)
 		(fp_line
-			(start -0.237258 0.5225)
-			(end 0.237258 0.5225)
+			(start -0.237258 -0.5225)
+			(end 0.237258 -0.5225)
 			(stroke
 				(width 0.12)
@@
 		)
 		(fp_line
-			(start 1.48 -0.73)
-			(end 1.48 0.73)
+			(start -1.48 0.73)
+			(end -1.48 -0.73)
 			(stroke
 				(width 0.05)
@@
 		)
 		(fp_line
-			(start -1.48 -0.73)
-			(end 1.48 -0.73)
+			(start 1.48 0.73)
+			(end -1.48 0.73)
 			(stroke
 				(width 0.05)
@@
 		)
 		(fp_line
-			(start 1.48 0.73)
-			(end -1.48 0.73)
+			(start -1.48 -0.73)
+			(end 1.48 -0.73)
 			(stroke
 				(width 0.05)
@@
 		)
 		(fp_line
-			(start -1.48 0.73)
-			(end -1.48 -0.73)
+			(start 1.48 -0.73)
+			(end 1.48 0.73)
 			(stroke
 				(width 0.05)
@@
 		)
 		(fp_line
-			(start 0.8 -0.4125)
-			(end 0.8 0.4125)
+			(start -0.8 0.4125)
+			(end -0.8 -0.4125)
 			(stroke
 				(width 0.1)
@@
 		)
 		(fp_line
-			(start -0.8 -0.4125)
-			(end 0.8 -0.4125)
+			(start 0.8 0.4125)
+			(end -0.8 0.4125)
 			(stroke
 				(width 0.1)
@@
 		)
 		(fp_line
-			(start 0.8 0.4125)
-			(end -0.8 0.4125)
+			(start -0.8 -0.4125)
+			(end 0.8 -0.4125)
 			(stroke
 				(width 0.1)
@@
 		)
 		(fp_line
-			(start -0.8 0.4125)
-			(end -0.8 -0.4125)
+			(start 0.8 -0.4125)
+			(end 0.8 0.4125)
 			(stroke
 				(width 0.1)
@@
 		)
 		(pad "1" smd roundrect
-			(at -0.825 0 90)
+			(at -0.825 0 270)
 			(size 0.8 0.95)
 			(layers "F.Cu" "F.Mask" "F.Paste")
@@
 		)
 		(pad "2" smd roundrect
-			(at 0.825 0 90)
+			(at 0.825 0 270)
 			(size 0.8 0.95)
 			(layers "F.Cu" "F.Mask" "F.Paste")
@@
 	(footprint "LED_SMD:LED_0603_1608Metric"
 		(layer "F.Cu")
-		(at 160.909 96.901 -90)
+		(at 160.909 93.599 -90)
 		(descr "LED SMD 0603 (1608 Metric), square (rectangular) end terminal, IPC_7351 nominal, (Body size source: http://www.tortai-tech.com/upload/download/2011102023233369053.pdf), generated with kicad-footprint-generator")
 		(tags "LED")
@@
 			(layers "F.Cu" "F.Mask" "F.Paste")
 			(roundrect_rratio 0.25)
-			(net 88 "Net-(D1-K)")
+			(net 6 "RXD0")
 			(pinfunction "K")
 			(pintype "passive")
@@
 	(footprint "LED_SMD:LED_0603_1608Metric"
 		(layer "F.Cu")
-		(at 160.909 93.599 90)
+		(at 160.909 96.901 90)
 		(descr "LED SMD 0603 (1608 Metric), square (rectangular) end terminal, IPC_7351 nominal, (Body size source: http://www.tortai-tech.com/upload/download/2011102023233369053.pdf), generated with kicad-footprint-generator")
 		(tags "LED")
@@
 			(layers "F.Cu" "F.Mask" "F.Paste")
 			(roundrect_rratio 0.25)
-			(net 85 "Net-(D2-K)")
+			(net 7 "TXD0")
 			(pinfunction "K")
 			(pintype "passive")
@@
 			)
 		)
-		(property "LCSC" ""
+		(property "LCSC" "C2661571"
 			(at 0 0 0)
 			(unlocked yes)
@@
 		(sheetname "/")
 		(sheetfile "AiO-i2s-DAC.kicad_sch")
-		(attr smd exclude_from_bom dnp)
+		(attr smd dnp)
 		(fp_line
 			(start -0.162779 -0.51)
@@
 	)
 	(segment
-		(start 160.909 97.6885)
-		(end 159.1685 97.6885)
+		(start 159.2965 92.774)
+		(end 160.909 94.3865)
 		(width 0.2032)
 		(layer "F.Cu")
@@
 	)
 	(segment
-		(start 159.1685 97.6885)
-		(end 159.131 97.726)
+		(start 159.131 92.774)
+		(end 159.2965 92.774)
 		(width 0.2032)
 		(layer "F.Cu")
@@
 	)
 	(segment
-		(start 159.1685 92.8115)
-		(end 159.131 92.774)
+		(start 159.131 97.726)
+		(end 159.2965 97.726)
 		(width 0.2032)
 		(layer "F.Cu")
@@
 	)
 	(segment
-		(start 160.909 92.8115)
-		(end 159.1685 92.8115)
+		(start 159.2965 97.726)
+		(end 160.909 96.1135)
 		(width 0.2032)
 		(layer "F.Cu")
@@
 	)
 	(segment
+		(start 160.597744 90.990463)
+		(end 160.597744 92.500244)
+		(width 0.2032)
+		(layer "F.Cu")
+		(net 6)
+	)
+	(segment
+		(start 160.597744 92.500244)
+		(end 160.909 92.8115)
+		(width 0.2032)
+		(layer "F.Cu")
+		(net 6)
+	)
+	(segment
 		(start 157.353 90.932)
 		(end 157.353 92.071308)
@@
 	)
 	(segment
+		(start 161.798 98.806)
+		(end 161.798 98.5775)
+		(width 0.2032)
+		(layer "F.Cu")
+		(net 7)
+	)
+	(segment
+		(start 161.798 98.5775)
+		(end 160.909 97.6885)
+		(width 0.2032)
+		(layer "F.Cu")
+		(net 7)
+	)
+	(segment
 		(start 156.5852 92.3348)
 		(end 155.5096 92.3348)
@@
 	)
 	(segment
-		(start 161.5185 94.996)
-		(end 160.909 94.3865)
-		(width 0.2032)
-		(layer "F.Cu")
-		(net 85)
-	)
-	(segment
-		(start 162.777 94.996)
-		(end 161.5185 94.996)
-		(width 0.2032)
-		(layer "F.Cu")
-		(net 85)
-	)
-	(segment
 		(start 159.131 111.061)
 		(end 159.131 111.0488)
@@
 	)
 	(segment
-		(start 162.777 95.496)
-		(end 161.5265 95.496)
-		(width 0.2032)
-		(layer "F.Cu")
-		(net 88)
-	)
-	(segment
-		(start 161.5265 95.496)
-		(end 160.909 96.1135)
-		(width 0.2032)
-		(layer "F.Cu")
-		(net 88)
-	)
-	(segment

Commit message: CP2104 layout
Parts:
- removed U4: CP2102-GM, Package_DFN_QFN:QFN-28-1EP_5x5mm_P0.5mm_EP3.35x3.35mm
- added C19: 4.7uF 16V, Capacitor_SMD:C_0603_1608Metric, F.Cu at (162.5, 107.5)
- added JP4: CTS1, Jumper:SolderJumper-2_P1.3mm_Open_RoundedPad1.0x1.5mm, B.Cu at (165.0, 104.2)
- added U6: CP2104, Package_DFN_QFN:QFN-24-1EP_4x4mm_P0.5mm_EP2.6x2.6mm_ThermalVias, F.Cu at (166.0, 108.1)
- R23: value 22.1K 1% -> 24K 1%
- R24: value 47.5K 1% -> 47K 1%
Connections:
- net /CP2102-GM/D+ renamed /CP2104-F03-GM/D+
- net /CP2102-GM/D- renamed /CP2104-F03-GM/D-
Routing:
- net /CP2104-F03-GM/CTS: track 0.00 -> 7.61 mm, vias 0 -> 1
- net Net-(U6-VPP): track 0.00 -> 1.52 mm
- net Net-(U6-RXD): track 2.23 -> 3.00 mm
- net Net-(U6-TXD): track 2.24 -> 3.00 mm
- net AGND: vias 296 -> 293
Other:
- board text added: "CTS1"

Commit message: Repositioning
Parts:
- moved C19 0.13 mm to (162.7, 107.5)
Changed lines of the file:
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@@
 	(footprint "Capacitor_SMD:C_0603_1608Metric"
 		(layer "F.Cu")
-		(at 162.5346 107.5436 90)
+		(at 162.6616 107.5436 90)
 		(descr "Capacitor SMD 0603 (1608 Metric), square (rectangular) end terminal, IPC_7351 nominal, (Body size source: IPC-SM-782 page 76, https://www.pcb-3d.com/wordpress/wp-content/uploads/ipc-sm-782a_amendment_1_and_2.pdf), generated with kicad-footprint-generator")
 		(tags "capacitor")
@@
 	)
 	(segment
-		(start 162.543 108.327)
-		(end 162.5346 108.3186)
+		(start 162.67 108.327)
+		(end 162.6616 108.3186)
 		(width 0.2032)
 		(layer "F.Cu")
@@
 	(segment
 		(start 164.0515 108.327)
-		(end 162.543 108.327)
+		(end 162.67 108.327)
 		(width 0.2032)
 		(layer "F.Cu")
