File: pcbs/AiO-i2s-DAC/AiO-i2s-DAC.kicad_sch (KiCad schematic)
At the start: 64 parts, among them J1 UART1, J2 SJ-3524-SMT-TR, J3 Audio Out, J4 UART0, J7 Conn_01x02, Q3 BC818, Q4 MBT3904DW1, Q6 MBT3904DW1, U1 ESP32-WROVER-E, U2 AZ1117CH-3.3TRG1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

Commit message: Adding equivalent JLCPCB values
Parts:
- C1, C18, C22, C23, C25, C3, C8, C9: LCSC (none) -> C14663
- C16, C2, C6, C7: LCSC (none) -> C45783
- C17, C20: LCSC (none) -> C23630
- C21, C24, C26, C29: LCSC (none) -> C15850
- C27, C28: LCSC (none) -> C1604
- D5, D6: LCSC (none) -> C2286
- J1: now left out of the parts list
- J2: Arrow Part Number SJ-3524-SMT-TR -> (none); Mouser Part Number 490-SJ-3524-SMT-TR -> (none)
- J7: now not fitted; now left out of the parts list
- Q3: LCSC (none) -> C154797
- Q4, Q6: LCSC (none) -> C131781
- R12, R13, R14, R32, R33, R36, R37, R38, R39, R40, R7: LCSC (none) -> C25804
- R3, R4: LCSC (none) -> C23179
- R41: LCSC (none) -> C21189
- R5, R6: LCSC (none) -> C21190
- S1, S2: Mouser Part Number 612-TL3305BF260QG -> (none); Mouser Price/Stock https://www.mouser.co.uk/ProductDetail/E-Switch/TL3305BF260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 -> (none)
- U1: LCSC (none) -> C967023
- U2: LCSC (none) -> C6186
- U5: LCSC (none) -> C107671

Commit message: LCSC BOM Preparation
Parts:
- C1, C18, C22, C23, C25, C3, C8, C9: LCSC alt (none) -> C1591
- C16, C2, C6, C7: LCSC alt (none) -> C380336
- C17, C20: LCSC alt (none) -> C23630
- C21, C24, C26, C29: LCSC alt (none) -> C1713
- C27, C28: LCSC alt (none) -> C107082
- D5: LCSC alt (none) -> C157740
- D6: LCSC alt (none) -> C364560
- J2: LCSC alt (none) -> C2910529
- Q3: LCSC alt (none) -> C154797
- Q4, Q6: LCSC alt (none) -> C110150
- R12, R13, R14, R32, R33, R36, R37, R38, R39, R40, R7: LCSC alt (none) -> C2479067
- R3, R4: LCSC alt (none) -> C23179
- R41: LCSC alt (none) -> C21189
- R5, R6: LCSC alt (none) -> C22548
- S1, S2: LCSC alt (none) -> C412373
- U1: LCSC alt (none) -> C2973667
- U2: LCSC alt (none) -> C92102
- U5: LCSC alt (none) -> C107671

Commit message: Build prep
Parts:
- R3, R4: LCSC C23179 -> C114669

Commit message: UART0 LEDs correction
Parts:
- FB1: LCSC (none) -> C2661571; now in the parts list
Changed lines of the file:
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@@
 	(title_block
 		(title "AiO-i2s-DAC")
-		(date "2025-09-02")
-		(rev "0.1.6")
+		(date "2025-10-05")
+		(rev "0.1.7")
 		(company "Martin Roger")
 	)
@@
 		(unit 1)
 		(exclude_from_sim yes)
-		(in_bom no)
+		(in_bom yes)
 		(on_board yes)
 		(dnp yes)
@@
 			)
 		)
-		(property "LCSC" ""
+		(property "LCSC" "C2661571"
 			(at 34.29 138.43 0)
 			(effects
@@
 					(size 1.27 1.27)
 				)
+				(hide yes)
 			)
 		)
@@
 					(size 1.27 1.27)
 				)
+				(hide yes)
 			)
 		)

Commit message: Schematic AiO with CP2104
Other:
- sheet CP2102-GM renamed CP2104-F03-GM
- sheet CP2104-F03-GM: file CP2102-GM.kicad_sch -> CP2104-F03-GM.kicad_sch
Changed lines of the file:
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@@
 			(color 0 0 0 0.0000)
 		)
-		(property "Sheetname" "CP2102-GM"
-			(at 326.39 151.13 0)
+		(property "Sheetname" "CP2104-F03-GM"
+			(at 321.31 151.638 0)
 			(effects
 				(font
@@
 			)
 		)
-		(property "Sheetfile" "CP2102-GM.kicad_sch"
+		(property "Sheetfile" "CP2104-F03-GM.kicad_sch"
 			(at 341.63 160.02 90)
 			(effects

Commit message: CP2104 layout
Parts:
- added JP4: CTS1, Jumper:SolderJumper-2_P1.3mm_Open_RoundedPad1.0x1.5mm, symbol Jumper:SolderJumper_2_Open
Connections:
- net CP2104-F03-GM/CTS: now also JP4.1 (A)
- net GND: now also JP4.2 (B)
- no-connect marks 21 -> 20
Changed lines of the file:
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@@
 	)
 	(no_connect
-		(at 337.82 134.62)
-	)
-	(no_connect
 		(at 95.25 76.2)
 	)
@@
 	(wire
 		(pts
+			(xy 337.82 129.54) (xy 337.82 134.62)
+		)
+		(stroke
+			(width 0)
+			(type default)
+		)
+	)
+	(wire
+		(pts
 			(xy 314.96 226.06) (xy 314.96 228.6)
 		)
@@
 	(wire
 		(pts
+			(xy 337.82 120.65) (xy 337.82 121.92)
+		)
+		(stroke
+			(width 0)
+			(type default)
+		)
+	)
+	(wire
+		(pts
 			(xy 394.97 210.82) (xy 388.62 210.82)
 		)
@@
 	)
 	(symbol
+		(lib_id "Jumper:SolderJumper_2_Open")
+		(at 337.82 125.73 90)
+		(unit 1)
+		(exclude_from_sim yes)
+		(in_bom no)
+		(on_board yes)
+		(dnp no)
+		(fields_autoplaced yes)
+		(property "Reference" "JP4"
+			(at 340.36 124.4599 90)
+			(effects
+				(font
+					(size 1.27 1.27)
+				)
+				(justify right)
+			)
+		)
+		(property "Value" "CTS1"
+			(at 340.36 126.9999 90)
+			(effects
+				(font
+					(size 1.27 1.27)
+				)
+				(justify right)
+			)
+		)
+		(property "Footprint" "Jumper:SolderJumper-2_P1.3mm_Open_RoundedPad1.0x1.5mm"
+			(at 337.82 125.73 0)
+			(effects
+				(font
+					(size 1.27 1.27)
+				)
+				(hide yes)
+			)
+		)
+		(property "Datasheet" "~"
+			(at 337.82 125.73 0)
+			(effects
+				(font
+					(size 1.27 1.27)
+				)
+				(hide yes)
+			)
+		)
+		(property "Description" "Solder Jumper, 2-pole, open"
+			(at 337.82 125.73 0)
+			(effects
+				(font
+					(size 1.27 1.27)
+				)
+				(hide yes)
+			)
+		)
+		(pin "1"
+		)
+		(pin "2"
+		)
+		(instances
+			(project ""
+				(path "/473bba75-08f8-4c6c-a9b2-aa3e95e63a5e"
+					(reference "JP4")
+					(unit 1)
+				)
+			)
+		)
+	)
+	(symbol
 		(lib_id "Connector:TestPoint_Small")
 		(at 308.61 209.55 270)
@@
 					(unit 1)
 				)
+			)
+		)
+	)
+	(symbol
+		(lib_id "power:GND")
+		(at 337.82 120.65 180)
+		(unit 1)
+		(exclude_from_sim no)
+		(in_bom yes)
+		(on_board yes)
+		(dnp no)
+		(fields_autoplaced yes)
+		(property "Reference" "#PWR050"
+			(at 337.82 114.3 0)
+			(effects
+				(font
+					(size 1.27 1.27)
+				)
+				(hide yes)
+			)
+		)
+		(property "Value" "GND"
+			(at 337.82 115.57 0)
+			(effects
+				(font
+					(size 1.27 1.27)
+				)
+			)
+		)
+		(property "Footprint" ""
+			(at 337.82 120.65 0)
+			(effects
+				(font
+					(size 1.27 1.27)
+				)
+				(hide yes)
+			)
+		)
+		(property "Datasheet" ""
+			(at 337.82 120.65 0)
+			(effects
+				(font
+					(size 1.27 1.27)
+				)
+				(hide yes)
+			)
+		)
+		(property "Description" ""
+			(at 337.82 120.65 0)
+			(effects
+				(font
+					(size 1.27 1.27)
+				)
+			)
+		)
+		(pin "1"
+		)
+		(instances
+			(project "AiO-i2s-DAC"
+				(path "/473bba75-08f8-4c6c-a9b2-aa3e95e63a5e"
+					(reference "#PWR050")
+					(unit 1)
+				)
