File: pcbs/AiO-i2s-DAC/AiO-i2s-DAC.kicad_sch (KiCad schematic)
At the start: 64 parts, among them J1 UART1, J2 SJ-3524-SMT-TR, J3 Audio Out, J4 UART0, J7 Conn_01x02, Q3 BC818, Q4 MBT3904DW1, Q6 MBT3904DW1, U1 ESP32-WROVER-E, U2 AZ1117CH-3.3TRG1, U5 PCM5102A

Commit message: S3 insertion start
Parts:
- added D12, D13, D3, D4: 2.1V G 10mA, LED_SMD:LED_0603_1608Metric, symbol Device:LED_Small
- added DTR0, HPD1, RTS0: TestPoint_Small, TestPoint:TestPoint_Pad_D2.0mm, symbol Connector:TestPoint_Small
- added JP4: HPD bypass, Jumper:SolderJumper-2_P1.3mm_Open_RoundedPad1.0x1.5mm, symbol Jumper:SolderJumper_2_Bridged
- added JP5: CDC_SEL, Jumper:SolderJumper-3_P1.3mm_Bridged12_RoundedPad1.0x1.5mm, symbol Jumper:SolderJumper_3_Bridged12
- added R10, R11, R8, R9: 1K 1%, Resistor_SMD:R_0603_1608Metric, symbol Device:R_Small
- added R42, R43: 10K 1%, Resistor_SMD:R_0603_1608Metric, symbol Device:R_Small
- added U6: ESP32-S3, Package_DFN_QFN:QFN-56-1EP_7x7mm_P0.4mm_EP5.6x5.6mm, symbol PCM_Espressif:ESP32-S3
- JP1: now not fitted
Connections:
- net DCD is gone; now on net GND: J1.2 (Pin_2), JP1.2 (C)
- net +3.3V: now also R10.1, R11.1, R43.2, R8.1, R9.1
- net DTR0: now also DTR0.1, U6.11 (GPIO6/ADC1_CH5)
- net GND: now also U6.57 (GND)
- net RTS0: now also RTS0.1, U6.12 (GPIO7/ADC1_CH6)
- net RXD0: now also D3.1 (K), U6.23 (GPIO17/ADC2_CH6)
- net RXD1: now also D12.1 (K), U6.16 (GPIO11/ADC2_CH0)
- net TXD0: now also D4.1 (K), U6.24 (GPIO18/ADC2_CH7)
- net TXD1: now also D13.1 (K), U6.17 (GPIO12/ADC2_CH1)
- net at J2.TN: now also JP4.1 (A)
- net BOOT: now reaches C9.2, R32.1, R33.1, S1.1, S1.2
- net BOOT: now also JP5.3 (B)
- new net: JP5.2 (C), U6.22 (GPIO16/ADC2_CH5/XTAL_32K_N)
- new net: U6.55 (VDDA), U6.56 (VDDA)
- new net: D3.2 (A), R8.2
- new net: JP4.2 (B), R42.1
- new net: D12.2 (A), R10.2
- new net: D13.2 (A), R11.2
- new net: D4.2 (A), R9.2
- new net HP_DETECT: HPD1.1, JP5.1 (A), R42.2, R43.1
- new net VDD3P3: U6.2 (VDD3P3), U6.3 (VDD3P3)
- new net usb_dn: U6.25 (GPIO19/USB_D-/ADC2_CH8)
- new net usb_dp: U6.26 (GPIO20/USB_D+/ADC2_CH9)
- no-connect marks 21 -> 20
Other:
- moved on the sheet: C17, C18, C20, C27, C28, C29, J2, J3, R3, R4, U5

Commit message: Preliminary S3 version schematic and layout
Parts:
- removed DCD1, GND1: TestPoint_Small, TestPoint:TestPoint_Pad_D1.0mm, symbol Connector:TestPoint_Small
- removed J1: UART1, Connector_PinHeader_2.54mm:PinHeader_1x05_P2.54mm_Vertical, symbol Connector_Generic:Conn_01x05
- removed J4: UART0, Connector_PinHeader_2.54mm:PinHeader_1x04_P2.54mm_Vertical, symbol Connector_Generic:Conn_01x04
- removed J7: Conn_01x02, Connector_PinHeader_2.54mm:PinHeader_1x02_P2.54mm_Vertical, symbol Connector_Generic:Conn_01x02
- removed JP1: ActDCD, Jumper:SolderJumper-3_P1.3mm_Bridged12_RoundedPad1.0x1.5mm, symbol Jumper:SolderJumper_3_Bridged12
- removed JP5: CDC_SEL, Jumper:SolderJumper-3_P1.3mm_Bridged12_RoundedPad1.0x1.5mm, symbol Jumper:SolderJumper_3_Bridged12
- removed R42: 10K 1%, Resistor_SMD:R_0603_1608Metric, symbol Device:R_Small
- removed U6: ESP32-S3, Package_DFN_QFN:QFN-56-1EP_7x7mm_P0.4mm_EP5.6x5.6mm, symbol PCM_Espressif:ESP32-S3
- added C30: 0.1uF 50V, Capacitor_SMD:C_0603_1608Metric, symbol Device:C_Small
- added C31: 10uF 16V, Capacitor_SMD:C_0805_2012Metric, symbol Device:C_Small
- added D11, D14: 1N5819HW-7-F, DIY:SOD3716X145N, symbol DIY:1N5819HW-7-F
- added JP7: BOOT Bypass, Jumper:SolderJumper-2_P1.3mm_Bridged_RoundedPad1.0x1.5mm, symbol Jumper:SolderJumper_2_Bridged
- added Q1: 2N7002, Package_TO_SOT_SMD:SOT-23, symbol Transistor_FET:2N7002
- added R15: 1K 1%, Resistor_SMD:R_0603_1608Metric, symbol Device:R_Small
- added R44, R49, R50: 10K 1%, Resistor_SMD:R_0603_1608Metric, symbol Device:R_Small
- added R45, R46, R47, R48: 0R, Resistor_SMD:R_0603_1608Metric, symbol Device:R_Small
- added S3: S3_BOOT, DIY:TL3305BF260QG, symbol DIY:TL3305BF260QG
- added TP1: 3V3, TestPoint:TestPoint_Pad_D2.0mm, symbol Connector:TestPoint_Small
- added TP2: RXD1, TestPoint:TestPoint_Pad_D2.0mm, symbol Connector:TestPoint_Small
- added TP3: TXD1, TestPoint:TestPoint_Pad_D2.0mm, symbol Connector:TestPoint_Small
- added TP4: DCD, TestPoint:TestPoint_Pad_D2.0mm, symbol Connector:TestPoint_Small
- added TP5: GND, TestPoint:TestPoint_Pad_D2.0mm, symbol Connector:TestPoint_Small
- added TP6: RXD0, TestPoint:TestPoint_Pad_D2.0mm, symbol Connector:TestPoint_Small
- added TP7: TXD0, TestPoint:TestPoint_Pad_D2.0mm, symbol Connector:TestPoint_Small
- added U7: ESP32-S3-MINI-1U-Nx, PCM_Espressif:ESP32-S3-MINI-1U, symbol RF_Module:ESP32-S3-MINI-1U
- FB1: now left out of the parts list
- J2: LCSC (none) -> C2910529; Manufacturer_Name Same Sky -> Korean HRO Parts Elec; Manufacturer_Part_Number SJ-3524-SMT-TR -> PJ-328-4A
- JP4: footprint Jumper:SolderJumper-2_P1.3mm_Open_RoundedPad1.0x1.5mm -> Jumper:SolderJumper-2_P1.3mm_Bridged_RoundedPad1.0x1.5mm
- S1: value TL3305BF260QG -> ESP_BOOT; LCSC (none) -> C412373; Manufacturer_Name E-Switch -> Shou Han; Manufacturer_Part_Number TL3305BF260QG -> TS4550TP
- S2: value TL3305BF260QG -> ESP_RESET; LCSC (none) -> C412373; Manufacturer_Name E-Switch -> Shou Han; Manufacturer_Part_Number TL3305BF260QG -> TS4550TP
- TP10: renamed from RTS0; value TestPoint_Small -> RTS 0; now left out of the parts list
- TP11: renamed from 3V1; value TestPoint_Small -> 3V3
- TP12: renamed from 5V1; value TestPoint_Small -> 5V
- TP13: renamed from HPD1; value TestPoint_Small -> HP detect; now left out of the parts list
- TP8: renamed from VBUS1; value TestPoint_Small -> VBUS
- TP9: renamed from DTR0; value TestPoint_Small -> DTR 0; now left out of the parts list
Connections:
- net IO5 is gone; now on net WSEL: U1.29 (GPIO5)
- net +3.3V: now also R45.1, R46.2, R50.2, TP1.1; no longer R43.2
- net BCLK: now also U1.31 (GPIO19); no longer U1.12 (ADC2_CH7/GPIO27)
- net BOOT: now also JP7.1 (A)
- net DIN: now also U1.30 (GPIO18); no longer U1.11 (DAC_2/ADC2_CH9/GPIO26)
- net DTR0: now also U7.17 (IO13)
- net GND: now also C30.1, C31.2, D11.2, Q1.2 (S), R44.1, R49.1, S3.1, S3.2, TP5.1, U7.1 (GND), U7.2 (GND), U7.42 (GND), U7.43 (GND), U7.46 (GND), U7.47 (GND), U7.48 (GND), U7.49 (GND), U7.50 (GND), U7.51 (GND), U7.52 (GND), U7.53 (GND), U7.54 (GND), U7.55 (GND), U7.56 (GND), U7.57 (GND), U7.58 (GND), U7.59 (GND), U7.60 (GND), U7.61 (GND), U7.62 (GND), U7.63 (GND), U7.64 (GND), U7.65 (GND)
- net RTS0: now also U7.16 (IO12)
- net RXD0: now also TP6.1, U7.8 (IO4)
- net RXD1: now also U1.36 (GPIO22), TP2.1, U7.6 (IO2); no longer U1.31 (GPIO19)
- net TXD0: now also TP7.1, U7.7 (IO3)
- net TXD1: now also U1.37 (GPIO23), TP3.1, U7.5 (IO1); no longer U1.33 (GPIO21)
- net WSEL: no longer U1.10 (DAC_1/ADC2_CH8/GPIO25)
- net at JP4.2 (B): now also D14.1
- net ~{BT_ST}: now reaches U1.16 (MTCK/GPIO13/ADC2_CH4)
- net ~{BT_ST}: now also D6.1 (K)
- net HP_DETECT renamed ~{HP_DETECT}
- net ~{HP_DETECT}: now also D11.1, D14.2, Q1.3 (D), U7.20 (IO16)
- removed net IO18: D6.1 (K), U1.30 (GPIO18)
- new net: C30.2, C31.1, R45.2, U7.3 (3V3)
- new net: S3.3, S3.4, U7.4 (IO0)
- new net: R46.1, U7.45 (EN)
- new net: JP7.2 (B), R15.1
- new net: Q1.1 (G), R15.2, R49.2
- new net: R43.2, R50.1
- new net DCD: R44.2, TP4.1, U1.33 (GPIO21), U7.9 (IO5)
- new net USBD+: R48.2, U7.24 (USB_D+)
- new net USBD-: R47.2, U7.23 (USB_D-)
- new net USB_DN: R47.1
- new net USB_DP: R48.1
- no-connect marks 20 -> 40
Other:
- sheet USB C 0 renamed USB C
- removed sheet CP2102-GM
- removed sheet CP2102_0
- removed sheet USB C 1
- sheet USB C ports: added DN, DP; removed USB_DN, USB_DP
- moved on the sheet: C16, C17, C18, C20, C21, C22, C23, C24, C25, C26, C27, C28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
