File: pcbs/AiO-i2s-DAC/CP2104-F03-GM.kicad_sch (KiCad schematic)
At the start: 13 parts, among them U6 CP2104

Commit message: A1S updated to CP2104
Version numbers also updated
Other:
- title: AiO-i2s-DAC -> CP2104
Changed lines of the file:
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@@
 	(paper "A4")
 	(title_block
-		(title "AiO-i2s-DAC")
-		(date "2025-10-05")
-		(rev "0.1.7")
+		(title "CP2104")
+		(date "2025-10-22")
+		(rev "0.2.0")
 		(company "Martin Roger")
 	)
