File: pcbs/a1s-mini/CP2102.kicad_sch (KiCad schematic)
At the start: 8 parts, among them U3 CP2102N-Axx-xQFN28

Commit message: Starting A1S Mini, teardrops on sandwhich
Parts:
- C8: value 0.1uF -> 0.1uF 50V; footprint (none) -> Capacitor_SMD:C_0805_2012Metric; Manufacturer_Name (none) -> YAGEO; Manufacturer_Part_Number (none) -> CC0805KRX7R9BB104
- C8: footprint (none) -> Capacitor_SMD:C_0805_2012Metric; Manufacturer_Name (none) -> KEMET; Manufacturer_Part_Number (none) -> C0805C106K8PACTU
- R15: renamed from R13; footprint (none) -> Resistor_SMD:R_0805_2012Metric; Manufacturer_Name (none) -> StackPole Electronics; Manufacturer_Part_Number (none) -> RMCF0805FT22K1
- R16: renamed from R12; footprint (none) -> Resistor_SMD:R_0805_2012Metric; Manufacturer_Name (none) -> StackPole Electronics; Manufacturer_Part_Number (none) -> RMCF0805FT47K5
- R4: footprint (none) -> Resistor_SMD:R_0805_2012Metric; Manufacturer_Name (none) -> YAGEO; Manufacturer_Part_Number (none) -> RC0805JR-070RL
- R4: footprint (none) -> Resistor_SMD:R_0805_2012Metric; Manufacturer_Name (none) -> StackPole Electronics; Manufacturer_Part_Number (none) -> RMCF0805FT2K00
- U3: value CP2102N-Axx-xQFN28 -> CP2102N; Manufacturer_Name (none) -> Silicon Labs; Manufacturer_Part_Number (none) -> CP2102N-A02-GQFN28R
Connections:
- net SUSPEND: no longer names the net of U3.12 (SUSPEND)
- net ~{RST}: no longer names the net of R4.2, U3.9 (~{RST})
- net ~{SUSPEND}: no longer names the net of U3.11 (~{SUSPEND})
- no-connect marks 9 -> 12

Commit message: Corrections and PCB layout
Parts:
- C8: footprint Capacitor_SMD:C_0805_2012Metric -> Capacitor_SMD:C_0603_1608Metric; Manufacturer_Name YAGEO -> Samsung Electro-Mechanics; Manufacturer_Part_Number CC0805KRX7R9BB104 -> CL10B104KB8NNNC
- C8: value 10uF -> 10uF 10V; footprint Capacitor_SMD:C_0805_2012Metric -> Capacitor_SMD:C_0603_1608Metric; Manufacturer_Name KEMET -> Samsung Electro-Mechanics; Manufacturer_Part_Number C0805C106K8PACTU -> CL10A106KP8NNNC
- R15: value 22.1K -> 22.1K 1%; footprint Resistor_SMD:R_0805_2012Metric -> Resistor_SMD:R_0603_1608Metric; Manufacturer_Part_Number RMCF0805FT22K1 -> RMCF0603FT22K1
- R16: value 47.5K -> 47.5K 1%; footprint Resistor_SMD:R_0805_2012Metric -> Resistor_SMD:R_0603_1608Metric; Manufacturer_Name StackPole Electronics -> Panasonic Electronic Components; Manufacturer_Part_Number RMCF0805FT47K5 -> ERJ-3EKF4752V
- R4: footprint Resistor_SMD:R_0805_2012Metric -> Resistor_SMD:R_0603_1608Metric; Manufacturer_Name YAGEO -> StackPole Electronics; Manufacturer_Part_Number RC0805JR-070RL -> RMCF0603ZT0R00
- R4: value 2K -> 2K 1%; footprint Resistor_SMD:R_0805_2012Metric -> Resistor_SMD:R_0603_1608Metric; Manufacturer_Part_Number RMCF0805FT2K00 -> RMCF0603FT2K00
Changed lines of the file:
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@@
       (effects (font (size 1.27 1.27)) (justify right))
     )
-    (property "Footprint" "Capacitor_SMD:C_0805_2012Metric" (at 139.7 60.96 0)
-      (effects (font (size 1.27 1.27)) hide)
-    )
-    (property "Datasheet" "https://www.yageo.com/upload/media/product/productsearch/datasheet/mlcc/UPY-GPHC_X7R_6.3V-to-250V_24.pdf" (at 139.7 60.96 0)
-      (effects (font (size 1.27 1.27)) hide)
-    )
-    (property "Description" "CAP CER 0.1UF 50V X7R 0805" (at 139.7 60.96 0)
-      (effects (font (size 1.27 1.27)) hide)
-    )
-    (property "Manufacturer_Name" "YAGEO" (at 139.7 60.96 0)
-      (effects (font (size 1.27 1.27)) hide)
-    )
-    (property "Manufacturer_Part_Number" "CC0805KRX7R9BB104" (at 139.7 60.96 0)
+    (property "Footprint" "Capacitor_SMD:C_0603_1608Metric" (at 139.7 60.96 0)
+      (effects (font (size 1.27 1.27)) hide)
+    )
+    (property "Datasheet" "https://mm.digikey.com/Volume0/opasdata/d220001/medias/docus/609/CL10B104KB8NNNC_Spec.pdf" (at 139.7 60.96 0)
+      (effects (font (size 1.27 1.27)) hide)
+    )
+    (property "Description" "CAP CER 0.1UF 50V X7R 0603" (at 139.7 60.96 0)
+      (effects (font (size 1.27 1.27)) hide)
+    )
+    (property "Manufacturer_Name" "Samsung Electro-Mechanics" (at 139.7 60.96 0)
+      (effects (font (size 1.27 1.27)) hide)
+    )
+    (property "Manufacturer_Part_Number" "CL10B104KB8NNNC" (at 139.7 60.96 0)
       (effects (font (size 1.27 1.27)) hide)
     )
@@
       (effects (font (size 1.27 1.27)))
     )
-    (property "Footprint" "Resistor_SMD:R_0805_2012Metric" (at 182.88 76.2 0)
-      (effects (font (size 1.27 1.27)) hide)
-    )
-    (property "Datasheet" "https://www.yageo.com/upload/media/product/products/datasheet/rchip/PYu-RC_Group_51_RoHS_L_12.pdf" (at 182.88 76.2 0)
-      (effects (font (size 1.27 1.27)) hide)
-    )
-    (property "Description" "RES 0 OHM JUMPER 1/8W 0805" (at 182.88 76.2 0)
-      (effects (font (size 1.27 1.27)) hide)
-    )
-    (property "Manufacturer_Name" "YAGEO" (at 182.88 76.2 0)
-      (effects (font (size 1.27 1.27)) hide)
-    )
-    (property "Manufacturer_Part_Number" "RC0805JR-070RL" (at 182.88 76.2 0)
+    (property "Footprint" "Resistor_SMD:R_0603_1608Metric" (at 182.88 76.2 0)
+      (effects (font (size 1.27 1.27)) hide)
+    )
+    (property "Datasheet" "https://www.seielect.com/catalog/sei-rmcf_rmcp.pdf" (at 182.88 76.2 0)
+      (effects (font (size 1.27 1.27)) hide)
+    )
+    (property "Description" "RES 0 OHM JUMPER 1/10W 0603" (at 182.88 76.2 0)
+      (effects (font (size 1.27 1.27)) hide)
+    )
+    (property "Manufacturer_Name" "StackPole Electronics" (at 182.88 76.2 0)
+      (effects (font (size 1.27 1.27)) hide)
+    )
+    (property "Manufacturer_Part_Number" "RMCF0603ZT0R00" (at 182.88 76.2 0)
       (effects (font (size 1.27 1.27)) hide)
     )
@@
       (effects (font (size 1.27 1.27)) (justify right))
     )
-    (property "Value" "10uF" (at 137.8014 50.8 0)
+    (property "Value" "10uF 10V" (at 137.8014 50.8 0)
       (effects (font (size 1.27 1.27)) (justify right))
     )
-    (property "Footprint" "Capacitor_SMD:C_0805_2012Metric" (at 139.7 48.26 0)
-      (effects (font (size 1.27 1.27)) hide)
-    )
-    (property "Datasheet" "https://search.kemet.com/download/datasheet/C0805C106K8PAC7800" (at 139.7 48.26 0)
-      (effects (font (size 1.27 1.27)) hide)
-    )
-    (property "Description" "CAP CER 10UF 10V X5R 0805" (at 139.7 48.26 0)
-      (effects (font (size 1.27 1.27)) hide)
-    )
-    (property "Manufacturer_Name" "KEMET" (at 139.7 48.26 0)
-      (effects (font (size 1.27 1.27)) hide)
-    )
-    (property "Manufacturer_Part_Number" "C0805C106K8PACTU" (at 139.7 48.26 0)
+    (property "Footprint" "Capacitor_SMD:C_0603_1608Metric" (at 139.7 48.26 0)
+      (effects (font (size 1.27 1.27)) hide)
+    )
+    (property "Datasheet" "https://mm.digikey.com/Volume0/opasdata/d220001/medias/docus/43/CL10A106KP8NNNC_Spec.pdf" (at 139.7 48.26 0)
+      (effects (font (size 1.27 1.27)) hide)
+    )
+    (property "Description" "CAP CER 10UF 10V X5R 0603" (at 139.7 48.26 0)
+      (effects (font (size 1.27 1.27)) hide)
+    )
+    (property "Manufacturer_Name" "Samsung Electro-Mechanics" (at 139.7 48.26 0)
+      (effects (font (size 1.27 1.27)) hide)
+    )
+    (property "Manufacturer_Part_Number" "CL10A106KP8NNNC" (at 139.7 48.26 0)
       (effects (font (size 1.27 1.27)) hide)
     )
@@
       (effects (font (size 1.27 1.27)))
     )
-    (property "Value" "22.1K" (at 107.95 83.82 90)
-      (effects (font (size 1.27 1.27)))
-    )
-    (property "Footprint" "Resistor_SMD:R_0805_2012Metric" (at 107.95 86.36 0)
+    (property "Value" "22.1K 1%" (at 107.95 83.82 90)
+      (effects (font (size 1.27 1.27)))
+    )
+    (property "Footprint" "Resistor_SMD:R_0603_1608Metric" (at 107.95 86.36 0)
       (effects (font (size 1.27 1.27)) hide)
     )
@@
       (effects (font (size 1.27 1.27)) hide)
     )
-    (property "Description" "RES 22.1K OHM 1% 1/8W 0805" (at 107.95 86.36 90)
+    (property "Description" "RES 22.1K OHM 1% 1/10W 0603" (at 107.95 86.36 90)
       (effects (font (size 1.27 1.27)) hide)
     )
@@
       (effects (font (size 1.27 1.27)) hide)
     )
-    (property "Manufacturer_Part_Number" "RMCF0805FT22K1" (at 107.95 86.36 0)
+    (property "Manufacturer_Part_Number" "RMCF0603FT22K1" (at 107.95 86.36 0)
       (effects (font (size 1.27 1.27)) hide)
     )
@@
       (effects (font (size 1.27 1.27)))
     )
-    (property "Footprint" "Resistor_SMD:R_0805_2012Metric" (at 173.99 73.66 0)
-      (effects (font (size 1.27 1.27)) hide)
-    )
-    (property "Datasheet" "https://www.yageo.com/upload/media/product/products/datasheet/rchip/PYu-RC_Group_51_RoHS_L_12.pdf" (at 173.99 73.66 0)
-      (effects (font (size 1.27 1.27)) hide)
-    )
-    (property "Description" "RES 0 OHM JUMPER 1/8W 0805" (at 173.99 73.66 0)
-      (effects (font (size 1.27 1.27)) hide)
-    )
-    (property "Manufacturer_Name" "YAGEO" (at 173.99 73.66 0)
-      (effects (font (size 1.27 1.27)) hide)
-    )
-    (property "Manufacturer_Part_Number" "RC0805JR-070RL" (at 173.99 73.66 0)
+    (property "Footprint" "Resistor_SMD:R_0603_1608Metric" (at 173.99 73.66 0)
+      (effects (font (size 1.27 1.27)) hide)
+    )
+    (property "Datasheet" "https://www.seielect.com/catalog/sei-rmcf_rmcp.pdf" (at 173.99 73.66 0)
+      (effects (font (size 1.27 1.27)) hide)
+    )
+    (property "Description" "RES 0 OHM JUMPER 1/10W 0603" (at 173.99 73.66 0)
+      (effects (font (size 1.27 1.27)) hide)
+    )
+    (property "Manufacturer_Name" "StackPole Electronics" (at 173.99 73.66 0)
+      (effects (font (size 1.27 1.27)) hide)
+    )
+    (property "Manufacturer_Part_Number" "RMCF0603ZT0R00" (at 173.99 73.66 0)
       (effects (font (size 1.27 1.27)) hide)
     )
@@
       (effects (font (size 1.27 1.27)))
     )
-    (property "Value" "2K" (at 127 76.2 90)
-      (effects (font (size 1.27 1.27)))
-    )
-    (property "Footprint" "Resistor_SMD:R_0805_2012Metric" (at 127 73.66 0)
+    (property "Value" "2K 1%" (at 127 76.2 90)
+      (effects (font (size 1.27 1.27)))
+    )
+    (property "Footprint" "Resistor_SMD:R_0603_1608Metric" (at 127 73.66 0)
       (effects (font (size 1.27 1.27)) hide)
     )
@@
       (effects (font (size 1.27 1.27)) hide)
     )
-    (property "Description" "RES 2K OHM 1% 1/8W 0805" (at 127 73.66 0)
+    (property "Description" "RES 2K OHM 1% 1/10W 0603" (at 127 73.66 0)
       (effects (font (size 1.27 1.27)) hide)
     )
@@
       (effects (font (size 1.27 1.27)) hide)
     )
-    (property "Manufacturer_Part_Number" "RMCF0805FT2K00" (at 127 73.66 0)
+    (property "Manufacturer_Part_Number" "RMCF0603FT2K00" (at 127 73.66 0)
       (effects (font (size 1.27 1.27)) hide)
     )
@@
       (effects (font (size 1.27 1.27)) (justify left))
     )
-    (property "Value" "47.5K" (at 115.57 97.155 0)
+    (property "Value" "47.5K 1%" (at 115.57 97.155 0)
       (effects (font (size 1.27 1.27)) (justify left))
     )
-    (property "Footprint" "Resistor_SMD:R_0805_2012Metric" (at 113.03 95.25 0)
-      (effects (font (size 1.27 1.27)) hide)
-    )
-    (property "Datasheet" "https://www.seielect.com/catalog/sei-rmcf_rmcp.pdf" (at 113.03 95.25 0)
-      (effects (font (size 1.27 1.27)) hide)
-    )
-    (property "Description" "RES 47.5K OHM 1% 1/8W 0805" (at 113.03 95.25 0)
-      (effects (font (size 1.27 1.27)) hide)
-    )
-    (property "Manufacturer_Name" "StackPole Electronics" (at 113.03 95.25 0)
-      (effects (font (size 1.27 1.27)) hide)
-    )
-    (property "Manufacturer_Part_Number" "RMCF0805FT47K5" (at 113.03 95.25 0)
-      (effects (font (size 1.27 1.27)) hide)
-    )
+    (property "Footprint" "Resistor_SMD:R_0603_1608Metric" (at 113.03 95.25 0)
+      (effects (font (size 1.27 1.27)) hide)
+    )
+    (property "Datasheet" "https://industrial.panasonic.com/cdbs/www-data/pdf/RDA0000/AOA0000C304.pdf" (at 113.03 95.25 0)
+      (effects (font (size 1.27 1.27)) hide)
+    )
+    (property "Description" "RES SMD 47.5K OHM 1% 1/10W 0603" (at 113.03 95.25 0)
+      (effects (font (size 1.27 1.27)) hide)
+    )
+    (property "Manufacturer_Name" "Panasonic Electronic Components" (at 113.03 95.25 0)
+      (effects (font (size 1.27 1.27)) hide)
+    )
+    (property "Manufacturer_Part_Number" "ERJ-3EKF4752V" (at 113.03 95.25 0)
+      (effects (font (size 1.27 1.27)) hide)
+    )

Commit message: PCB layout update
Parts:
- added D1, D2: 2.1V G 10mA, LED_SMD:LED_0603_1608Metric, symbol Device:LED_Small
- added R1, R2: 1K 1%, Resistor_SMD:R_0603_1608Metric, symbol Device:R_Small
Connections:
- net REGIN: now also R1.1, R2.1
- net at U3.18 (~{RXT}/GPIO.1): now also D2.1 (K)
- net at U3.19 (~{TXT}/GPIO.0): now also D1.1 (K)
- new net: D1.2 (A), R1.2
- new net: D2.2 (A), R2.2
- no-connect marks 12 -> 10
Other:
- moved on the sheet: R4

Commit message: A1S Mini quote PCBWay
Parts:
- C8, D1, D2, R1, R15, R16, R2, R4, U3: Type (none) -> SMD
Other:
- company: (none) -> Martin Roger
Changed lines of the file:
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@@
   (title_block
     (title "CP2102 28Pin Auxiliary circuit")
-    (date "2025-02-22")
-    (rev "0.1")
+    (date "2025-03-01")
+    (rev "0.2.0")
+    (company "Martin Roger")
   )
   (junction (at 142.24 58.42) (diameter 0) (color 0 0 0 0)
@@
       (effects (font (size 1.27 1.27)) hide)
     )
+    (property "Instructions/Notes" "" (at 203.2 100.33 0)
+      (effects (font (size 1.27 1.27)) hide)
+    )
+    (property "Type" "SMD" (at 203.2 100.33 0)
+      (effects (font (size 1.27 1.27)) hide)
+    )
     (pin "1")
     (pin "2")
@@
     )
     (property "Manufacturer_Part_Number" "CL10B104KB8NNNC" (at 139.7 60.96 0)
+      (effects (font (size 1.27 1.27)) hide)
+    )
+    (property "Instructions/Notes" "" (at 139.7 60.96 0)
+      (effects (font (size 1.27 1.27)) hide)
+    )
+    (property "Type" "SMD" (at 139.7 60.96 0)
       (effects (font (size 1.27 1.27)) hide)
     )
@@
       (effects (font (size 1.27 1.27)) hide)
     )
+    (property "Instructions/Notes" "" (at 195.58 110.49 0)
+      (effects (font (size 1.27 1.27)) hide)
+    )
+    (property "Type" "SMD" (at 195.58 110.49 0)
+      (effects (font (size 1.27 1.27)) hide)
+    )
     (pin "1")
     (pin "2")
@@
       (effects (font (size 1.27 1.27)) hide)
     )
+    (property "Instructions/Notes" "" (at 195.58 100.33 0)
+      (effects (font (size 1.27 1.27)) hide)
+    )
+    (property "Type" "SMD" (at 195.58 100.33 0)
+      (effects (font (size 1.27 1.27)) hide)
+    )
     (pin "1")
     (pin "2")
@@
       (effects (font (size 1.27 1.27)) hide)
     )
+    (property "Instructions/Notes" "" (at 185.42 80.01 0)
+      (effects (font (size 1.27 1.27)) hide)
+    )
+    (property "Type" "SMD" (at 185.42 80.01 0)
+      (effects (font (size 1.27 1.27)) hide)
+    )
     (pin "1")
     (pin "2")
@@
       (effects (font (size 1.27 1.27)) hide)
     )
+    (property "Instructions/Notes" "" (at 139.7 48.26 0)
+      (effects (font (size 1.27 1.27)) hide)
+    )
+    (property "Type" "SMD" (at 139.7 48.26 0)
+      (effects (font (size 1.27 1.27)) hide)
+    )
     (pin "1")
     (pin "2")
@@
       (effects (font (size 1.27 1.27)) hide)
     )
+    (property "Instructions/Notes" "" (at 107.95 86.36 0)
+      (effects (font (size 1.27 1.27)) hide)
+    )
+    (property "Type" "SMD" (at 107.95 86.36 0)
+      (effects (font (size 1.27 1.27)) hide)
+    )
     (pin "1")
     (pin "2")
@@
       (effects (font (size 1.27 1.27)) hide)
     )
+    (property "Instructions/Notes" "" (at 203.2 110.49 0)
+      (effects (font (size 1.27 1.27)) hide)
+    )
+    (property "Type" "SMD" (at 203.2 110.49 0)
+      (effects (font (size 1.27 1.27)) hide)
+    )
     (pin "1")
     (pin "2")
@@
     )
     (property "Manufacturer_Part_Number" "RMCF0603ZT0R00" (at 185.42 72.39 0)
+      (effects (font (size 1.27 1.27)) hide)
+    )
+    (property "Instructions/Notes" "" (at 185.42 72.39 0)
+      (effects (font (size 1.27 1.27)) hide)
+    )
+    (property "Type" "SMD" (at 185.42 72.39 0)
       (effects (font (size 1.27 1.27)) hide)
     )
@@
       (effects (font (size 1.27 1.27)) hide)
     )
+    (property "Instructions/Notes" "" (at 127 73.66 0)
+      (effects (font (size 1.27 1.27)) hide)
+    )
+    (property "Type" "SMD" (at 127 73.66 0)
+      (effects (font (size 1.27 1.27)) hide)
+    )
     (pin "1")
     (pin "2")
@@
       (effects (font (size 1.27 1.27)) hide)
     )
+    (property "Instructions/Notes" "" (at 113.03 95.25 0)
+      (effects (font (size 1.27 1.27)) hide)
+    )
+    (property "Type" "SMD" (at 113.03 95.25 0)
+      (effects (font (size 1.27 1.27)) hide)
+    )
     (pin "1")
     (pin "2")
@@
       (effects (font (size 1.27 1.27)) hide)
     )
+    (property "Instructions/Notes" "" (at 153.67 101.6 0)
+      (effects (font (size 1.27 1.27)) hide)
+    )
+    (property "Type" "SMD" (at 153.67 101.6 0)
+      (effects (font (size 1.27 1.27)) hide)
+    )

Commit message: Projects consistency update
Parts:
- renumbered C8 to C10, C8 to C11, R4 to R17, R4 to R18, R4 to R19
Other:
- title: CP2102 28Pin Auxiliary circuit -> A1S Mini Board
